Commit message: fixed lidar height and frame

File: urdf/wadribie.urdf.xacro (robot description, xacro)
@@ -9,5 +9,5 @@
   <link name="rplidar">
     <visual>
-      <origin xyz="0 0 0" rpy="0 0 ${- M_PI/2}" />
+      <origin xyz="0 0 -0.03" rpy="0 0 ${- M_PI/2}" />
       <geometry>
         <mesh filename="package://wadribie_robot/model/rplidar.stl"/>
@@ -21,5 +21,5 @@
     <child link="rplidar" />
     <parent link="base_link" />
-    <origin xyz="0 0 0.04" rpy="0 0 0" />
+    <origin xyz="0 0 0.07" rpy="0 0 0" />
   </joint>
 </robot>

Commit message: fixed hector slam configuration

File: urdf/wadribie.urdf.xacro (robot description, xacro)
@@ -7,5 +7,5 @@
   <xacro:property name="M_PI" value="3.14159265359"/>
   <xacro:include filename="$(find simplebot_driver)/urdf/simplebot.urdf.xacro" />
-  <link name="rplidar">
+  <link name="laser_link">
     <visual>
       <origin xyz="0 0 -0.03" rpy="0 0 ${- M_PI/2}" />
@@ -19,5 +19,5 @@
   </link>
    <joint name="rplidar_to_base_joint" type="fixed">
-    <child link="rplidar" />
+    <child link="laser_link" />
     <parent link="base_link" />
     <origin xyz="0 0 0.07" rpy="0 0 0" />
