Commit message: removed localization ground truth

File: wadribie_description/urdf/wadribie.urdf.xacro (robot description, xacro)
@@ -18,16 +18,9 @@
     </visual>
   </link>
-   <joint name="rplidar_to_base_joint" type="fixed">
+  <joint name="rplidar_to_base_joint" type="fixed">
     <child link="laser_link" />
     <parent link="base_link" />
     <origin xyz="0 0 0.07" rpy="0 0 0" />
   </joint>
-  <plugin name="p3d_base_controller" filename="libgazebo_ros_p3d.so">
-    <frameName>odom_combined</frameName>
-    <bodyName>base_link</bodyName>
-    <topicName>odom</topicName>
-    <updateRate>20.0</updateRate>
-    <gaussianNoise>0.01</gaussianNoise>
-  </plugin>
   <gazebo reference="laser_link">
     <sensor name="rplidar" type="ray">

Commit message: added imu to urdf

File: wadribie_description/urdf/wadribie.urdf.xacro (robot description, xacro)
@@ -7,4 +7,20 @@
   <xacro:property name="M_PI" value="3.14159265359"/>
   <xacro:include filename="$(find simplebot_driver)/urdf/simplebot.urdf.xacro" />
+  <link name="imu">
+    <visual>
+      <origin xyz="0 0 0.0" rpy="0 0 0" />
+      <geometry>
+        <box size="0.01 0.02 0.005"/>
+      </geometry>
+      <material name="darkblue" >
+        <color rgba="0.0 0.0 0.5 1" />
+      </material>
+    </visual>
+  </link>
+  <joint name="imu_to_base_joint" type="fixed">
+    <child link="imu" />
+    <parent link="base_link" />
+    <origin xyz="0 0 0.02" rpy="0 0 0" />
+  </joint>
   <link name="laser_link">
     <visual>
@@ -18,5 +34,5 @@
     </visual>
   </link>
-  <joint name="rplidar_to_base_joint" type="fixed">
+  <joint name="laser_to_base_joint" type="fixed">
     <child link="laser_link" />
     <parent link="base_link" />
